Commit message: Imported Kinova 6dof model into IsaacSim
- Improved URDF of the robot (revolute joints instead of continuous and added dynamic params)
- Added .usda files for the Kinova and for a simple testing scene

File: projects/vla_kinova_tabletop_isaac/isaacsim/worlds/kinova_gen3_6dof_2f85.urdf (robot description, URDF)
Before this commit: robot gen3, 21 links, 20 joints
Joints:
- joint robotiq_85_left_finger_tip_joint: limit (none) -> lower=-0.8 upper=0.0 effort=50 velocity=0.5; type continuous -> revolute
- joint robotiq_85_left_inner_knuckle_joint: limit (none) -> lower=0.0 upper=0.8 effort=50 velocity=0.5; type continuous -> revolute
- joint robotiq_85_right_finger_tip_joint: limit (none) -> lower=0.0 upper=0.8 effort=50 velocity=0.5; type continuous -> revolute
- joint robotiq_85_right_inner_knuckle_joint: limit (none) -> lower=-0.8 upper=0.0 effort=50 velocity=0.5; type continuous -> revolute
