Commit message: Improved gripper parallel mechanism, new vla_kinova_tabletop package
- Added 2 revolute joints to gripper (inner_knuckle_finger_tip_joints, left and right) to close the parallel mechanism loop, this was done to avoid having the gripper break down when grasping objects
- Removed joint drives from all the joints in the loop except for the left and right knuckle joints which are now the driving ones
- As ROS2 still tries to control all 6 original joints, I added a script node which filters the incoming messages and only outputs the left and right knuckle joint commands
- Excluded the left and right inner_knuckle_joints from the articulation: this was needed to avoid loop closure errors in the articulation, these are now the joints which accumulate the most error (the script node just ignores the incoming commands related to them)
- All these changes were done in the test.usda and kinova_tabletop.usda files, the original kinova_gen3_6dof_2f85.usda file still has the original 6 joints with the 6 joint drives
- Added vla_kinova_tabletop package with custom launchfiles and configuration for moveit/rviz/isaacsim setup
- Modified bootstrap_kinova_ws.bash to build using --symlink-install for convenience

Issues:
- There still seems to be conflict between the arm and gripper commands: the arm seems to block gripper commands
- General instability, might need joint drive tuning?

File: projects/vla_kinova_tabletop_isaac/ros2_ws/src/vla_kinova_tabletop/urdf/kinova_gen3_6dof_2f85.urdf (robot description, URDF)
Before this commit: robot kinova_gen3_6dof_2f85, 21 links, 20 joints
Joints:
- joint robotiq_85_left_finger_tip_joint: limit lower=-0.8 upper=0.0 effort=50 velocity=0.5 -> (none); type revolute -> continuous
- joint robotiq_85_left_inner_knuckle_joint: limit lower=0.0 upper=0.8 effort=50 velocity=0.5 -> (none); type revolute -> continuous
- joint robotiq_85_right_finger_tip_joint: limit lower=0.0 upper=0.8 effort=50 velocity=0.5 -> (none); type revolute -> continuous
- joint robotiq_85_right_inner_knuckle_joint: limit lower=-0.8 upper=0.0 effort=50 velocity=0.5 -> (none); type revolute -> continuous
