Commit message: Switched control point while teleoperating to a new tool_frame instead of end_effector_link
- New tool_frame in urdf/xacro defined as end_effector_link translated of 14 cm along z
- Updated the twist pose tracking node to compute error with respect to the control frame specified in the yaml
- The twist still needs to be sent relative to the end_effector_link so we transform it before sending it

File: projects/vla_kinova_tabletop_isaac/ros2_ws/src/vla_kinova_description/urdf/kortex_robot.xacro (robot description, xacro)
@@ -89,4 +89,14 @@
         use_internal_bus_gripper_comm="${use_internal_bus_gripper_comm}"
         moveit_active="${moveit_active}"/>
+      <!-- We added a new tool_frame, so that when we teleoperate we control this frame
+            instead of the end effector one, which is more intuitive in particular regarding orientation -->
+      <xacro:property name="grasp_offset" value="0.14"/>
+      <link name="${prefix}tool_frame"/>
+      <joint name="${prefix}tool_frame_joint" type="fixed">
+        <origin xyz="0 0 ${grasp_offset}" rpy="0 0 0" />
+        <parent link="${prefix}${last_arm_link}" />
+        <child link="${prefix}tool_frame" />
+        <axis xyz="0 0 0" />
+      </joint>
     </xacro:unless>
   </xacro:macro>

Commit message: Changed tool_frame to fingertips_frame to avoid confusion with firmware TOOL_FRAME and some cleanup)

File: projects/vla_kinova_tabletop_isaac/ros2_ws/src/vla_kinova_description/urdf/kortex_robot.xacro (robot description, xacro)
@@ -65,9 +65,9 @@
     <!-- If no gripper, define tool frame here -->
     <xacro:if value="${not gripper}">
-      <link name="${prefix}tool_frame"/>
-      <joint name="${prefix}tool_frame_joint" type="fixed">
+      <link name="${prefix}fingertips_frame"/>
+      <joint name="${prefix}fingertips_frame_joint" type="fixed">
         <origin xyz="0 0 0" rpy="0 0 0" />
         <parent link="${prefix}${last_arm_link}" />
-        <child link="${prefix}tool_frame" />
+        <child link="${prefix}fingertips_frame" />
         <axis xyz="0 0 0" />
       </joint>
@@ -89,12 +89,12 @@
         use_internal_bus_gripper_comm="${use_internal_bus_gripper_comm}"
         moveit_active="${moveit_active}"/>
-      <!-- We added a new tool_frame, so that when we teleoperate we control this frame
+      <!-- We added a new fingertips_frame, so that when we teleoperate we control this frame
             instead of the end effector one, which is more intuitive in particular regarding orientation -->
       <xacro:property name="grasp_offset" value="0.14"/>
-      <link name="${prefix}tool_frame"/>
-      <joint name="${prefix}tool_frame_joint" type="fixed">
+      <link name="${prefix}fingertips_frame"/>
+      <joint name="${prefix}fingertips_frame_joint" type="fixed">
         <origin xyz="0 0 ${grasp_offset}" rpy="0 0 0" />
         <parent link="${prefix}${last_arm_link}" />
-        <child link="${prefix}tool_frame" />
+        <child link="${prefix}fingertips_frame" />
         <axis xyz="0 0 0" />
       </joint>
